Commit message: 存在解析urdf后关节类型和连杆纹理文件导致的逻辑bug

File: src/robot_description/urdf/robot.urdf (robot description, URDF)
Before this commit: robot ur, 12 links, 11 joints
Links:
- added link base
Joints:
- added joint base_link-base_fixed_joint: type fixed, parent base_link, child base, origin xyz=0 0 0 rpy=0 0 3.141592653589793
