Commit message: update:  规划器测试代码

File: robot_resource/urdf/ur5e.urdf (robot description, URDF)
Before this commit: robot ur, 13 links, 12 joints
Links:
- link base_link_inertia: geometry collision mesh filename=package://fast_motion_planning/meshes/ur5e/collision/base.s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; visual mesh filename=package://fast_motion_planning/meshes/ur5e/visual/base.dae
- link forearm_link: geometry collision mesh filename=package://fast_motion_planning/meshes/ur5e/collision/forear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; visual mesh filename=package://fast_motion_planning/meshes/ur5e/visual/forearm.d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
- link shoulder_link: geometry collision mesh filename=package://fast_motion_planning/meshes/ur5e/collision/should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; visual mesh filename=package://fast_motion_planning/meshes/ur5e/visual/shoulder.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
- link upper_arm_link: geometry collision mesh filename=package://fast_motion_planning/meshes/ur5e/collision/uppera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; visual mesh filename=package://fast_motion_planning/meshes/ur5e/visual/upperarm.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
- link wrist_1_link: geometry collision mesh filename=package://fast_motion_planning/meshes/ur5e/collision/wrist1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; visual mesh filename=package://fast_motion_planning/meshes/ur5e/visual/wrist1.dae
- link wrist_2_link: geometry collision mesh filename=package://fast_motion_planning/meshes/ur5e/collision/wrist2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; visual mesh filename=package://fast_motion_planning/meshes/ur5e/visual/wrist2.dae
- link wrist_3_link: geometry collision mesh filename=package://fast_motion_planning/meshes/ur5e/collision/wrist3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; visual mesh filename=package://fast_motion_planning/meshes/ur5e/visual/wrist3.dae
